File: battery-lantern-v2/pcb/flicker_lamp.kicad_pcb (KiCad board)
At the start: 2 copper layers, 20.3 x 66 mm, 5 parts, among them U1 ATTINY13A-PU

Commit message: Battery lantern v2: PCB tweaks for v2A
- Silscreen LED holder glue area on both sides of PCB.
- Tabs on side for LED holder to sit on and align easily.
- Pull back copper pour near power connectors to avoid possibility of
  shorts through the solder mask by bent over wires.
- Widen slightly to avoid hot glue getting in power connector holes.
- Spread copper pours over bottom of PCB.
Parts:
- moved JLED1 2.54 mm to (160.0, 73.7)
Routing:
- net /VCC: track 69.3 -> 68.2 mm
- net /LED: track 42.5 -> 43.6 mm
- net /GND: track 58.6 -> 59.7 mm
Other:
- board size 20.3 x 66 mm -> 22.9 x 66 mm
- net class LED added: clearance 0.1524, trace_width 0.3048, via_dia 0.6858, via_drill 0.3302
- board text added: "Flicker lamp V2A 20200120"
- board text removed: "Flicker lamp V2 20191109"
Changed lines of the file:
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@@
     (links 12)
     (no_connects 0)
-    (area 140.079981 68.95998 162.660001 137.210001)
+    (area 140.079981 68.95998 165.150001 137.210001)
     (thickness 1.6)
-    (drawings 22)
-    (tracks 40)
+    (drawings 20)
+    (tracks 41)
     (zones 0)
     (modules 5)
@@
       (drillshape 0)
       (scaleselection 1)
-      (outputdirectory gerber/))
+      (outputdirectory gerber-20200120))
   )
   (net 0 "")
@@
     (uvia_dia 0.6858)
     (uvia_drill 0.3302)
-    (add_net /LED)
     (add_net /MISO)
     (add_net /MOSI)
@@
     (add_net /SCK)
     (add_net "Net-(U1-Pad2)")
+  )
+  (net_class LED ""
+    (clearance 0.1524)
+    (trace_width 0.3048)
+    (via_dia 0.6858)
+    (via_drill 0.3302)
+    (uvia_dia 0.6858)
+    (uvia_drill 0.3302)
+    (add_net /LED)
   )
   (net_class Power ""
@@
   )
   (module Socket_Strips:Socket_Strip_Straight_1x03_Pitch2.54mm (layer F.Cu)
-    (at 157.48 73.66 270)
+    (at 160.02 73.66 270)
     (descr "Through hole straight socket strip, 1x03, 2.54mm pitch, single row")
     (tags "Through hole socket strip THT 1x03 2.54mm single row")
@@
     )
   )
-  (gr_line (start 147.32 137.16) (end 162.56 137.16) (angle 90) (layer Edge.Cuts) (width 0.1))
+  (gr_line (start 165.1 137.16) (end 147.32 137.16) (angle 90) (layer Edge.Cuts) (width 0.1))
+  (gr_line (start 165.1 72.39) (end 165.1 81.788) (angle 90) (layer Edge.Cuts) (width 0.1))
+  (gr_line (start 165.1 81.788) (end 165.1 137.16) (angle 90) (layer Edge.Cuts) (width 0.1))
+  (gr_line (start 147.32 81.788) (end 147.32 104.14) (angle 90) (layer Edge.Cuts) (width 0.1))
+  (gr_line (start 149.86 81.788) (end 147.32 81.788) (angle 90) (layer Edge.Cuts) (width 0.1))
+  (gr_line (start 149.86 76.2) (end 149.86 81.788) (angle 90) (layer Edge.Cuts) (width 0.1))
   (gr_line (start 147.32 124.46) (end 147.32 137.16) (angle 90) (layer Edge.Cuts) (width 0.1))
-  (gr_line (start 162.56 124.46) (end 162.56 137.16) (angle 90) (layer Edge.Cuts) (width 0.1))
-  (gr_text "GND LED VCC" (at 154.94 75.438) (layer F.SilkS)
+  (gr_text "GND LED VCC" (at 157.48 75.438) (layer F.SilkS)
     (effects (font (size 0.762 0.762) (thickness 0.127)))
   )
-  (gr_line (start 147.32 72.39) (end 147.32 76.2) (angle 90) (layer Edge.Cuts) (width 0.1))
-  (gr_line (start 162.56 72.39) (end 162.56 76.2) (angle 90) (layer Edge.Cuts) (width 0.1))
-  (gr_line (start 162.56 76.2) (end 147.32 76.2) (angle 90) (layer F.SilkS) (width 0.2))
-  (gr_line (start 161.29 71.12) (end 162.56 72.39) (angle 90) (layer Edge.Cuts) (width 0.1))
-  (gr_line (start 148.59 71.12) (end 147.32 72.39) (angle 90) (layer Edge.Cuts) (width 0.1))
-  (gr_line (start 161.29 71.12) (end 148.59 71.12) (angle 90) (layer Edge.Cuts) (width 0.1))
-  (gr_line (start 147.32 76.2) (end 147.32 104.14) (angle 90) (layer Edge.Cuts) (width 0.1))
-  (gr_line (start 162.56 76.2) (end 162.56 104.14) (angle 90) (layer Edge.Cuts) (width 0.1))
-  (gr_line (start 147.32 104.14) (end 147.32 124.46) (angle 90) (layer F.SilkS) (width 0.2))
+  (gr_line (start 149.86 72.39) (end 149.86 76.2) (angle 90) (layer Edge.Cuts) (width 0.1))
+  (gr_line (start 163.83 71.12) (end 165.1 72.39) (angle 90) (layer Edge.Cuts) (width 0.1))
+  (gr_line (start 151.13 71.12) (end 149.86 72.39) (angle 90) (layer Edge.Cuts) (width 0.1))
+  (gr_line (start 163.83 71.12) (end 151.13 71.12) (angle 90) (layer Edge.Cuts) (width 0.1))
   (gr_line (start 142.24 109.22) (end 147.32 104.14) (angle 90) (layer Edge.Cuts) (width 0.1))
   (gr_line (start 142.24 119.38) (end 147.32 124.46) (angle 90) (layer Edge.Cuts) (width 0.1))
   (gr_line (start 142.24 109.22) (end 142.24 119.38) (angle 90) (layer Edge.Cuts) (width 0.1))
-  (gr_text "Flicker lamp\nV2 20191109" (at 156.21 104.902) (layer F.SilkS)
+  (gr_text "Flicker lamp\nV2A 20200120" (at 156.21 104.902) (layer F.SilkS)
     (effects (font (size 0.762 0.762) (thickness 0.127)))
   )
@@
     (effects (font (size 0.762 0.762) (thickness 0.127)) (justify left))
   )
-  (gr_line (start 162.56 104.14) (end 162.56 124.46) (angle 90) (layer Edge.Cuts) (width 0.1))
+  (segment (start 160.02 73.66) (end 160.02 76.2) (width 0.3048) (layer F.Cu) (net 1))
+  (segment (start 160.02 76.2) (end 160.02 107.95) (width 0.3048) (layer F.Cu) (net 1))
   (segment (start 160.02 107.95) (end 161.798 109.728) (width 0.3048) (layer F.Cu) (net 1))
-  (segment (start 160.02 107.95) (end 160.02 76.2) (width 0.3048) (layer F.Cu) (net 1))
-  (segment (start 160.02 76.2) (end 157.48 73.66) (width 0.3048) (layer F.Cu) (net 1))
   (segment (start 157.48 121.92) (end 155.702 123.698) (width 0.3048) (layer F.Cu) (net 1))
   (segment (start 146.05 118.11) (end 144.78 118.11) (width 0.3048) (layer F.Cu) (net 1))
@@
   (segment (start 161.798 120.65) (end 160.02 121.92) (width 0.3048) (layer F.Cu) (net 1))
   (segment (start 161.798 109.728) (end 161.798 120.65) (width 0.3048) (layer F.Cu) (net 1))
+  (segment (start 149.86 106.68) (end 157.48 99.06) (width 0.3048) (layer F.Cu) (net 2))
+  (segment (start 157.48 99.06) (end 157.48 73.66) (width 0.3048) (layer F.Cu) (net 2))
   (segment (start 152.4 113.03) (end 149.86 110.49) (width 0.3048) (layer F.Cu) (net 2))
-  (segment (start 154.94 101.6) (end 154.94 73.66) (width 0.3048) (layer F.Cu) (net 2))
-  (segment (start 149.86 106.68) (end 154.94 101.6) (width 0.3048) (layer F.Cu) (net 2))
   (segment (start 149.86 110.49) (end 149.86 106.68) (width 0.3048) (layer F.Cu) (net 2))
-  (segment (start 152.4 73.66) (end 149.86 76.2) (width 0.3048) (layer B.Cu) (net 3))
-  (segment (start 149.86 76.2) (end 149.86 113.03) (width 0.3048) (layer B.Cu) (net 3))
+  (segment (start 154.94 73.66) (end 154.94 101.6) (width 0.3048) (layer B.Cu) (net 3))
+  (segment (start 149.86 106.68) (end 149.86 113.03) (width 0.3048) (layer B.Cu) (net 3))
+  (segment (start 154.94 101.6) (end 149.86 106.68) (width 0.3048) (layer B.Cu) (net 3))
   (segment (start 152.4 115.57) (end 149.86 113.03) (width 0.3048) (layer B.Cu) (net 3))
   (segment (start 149.86 113.03) (end 147.32 110.49) (width 0.3048) (layer B.Cu) (net 3))
@@
   (segment (start 156.21 116.84) (end 156.21 116.84) (width 0.1524) (layer F.Cu) (net 9))
   (segment (start 157.48 110.49) (end 156.21 111.76) (width 0.1524) (layer F.Cu) (net 9))
-  (zone (net 1) (net_name /VCC) (layer F.Cu) (hatch edge 0.508)
+  (zone (net 0) (net_name "") (layer F.SilkS) (hatch full 0.508)
     (connect_pads (clearance 0.508))
     (min_thickness 0.254)
@@
     (polygon
       (pts
-        (xy 148.59 71.12) (xy 161.29 71.12) (xy 162.56 72.39) (xy 162.56 124.46) (xy 147.32 124.46)
-        (xy 142.24 119.38) (xy 142.24 109.22) (xy 147.32 104.14) (xy 147.32 72.39)
+        (xy 165.1 81.788) (xy 149.86 81.788) (xy 149.86 76.2) (xy 165.1 76.2)
       )
     )
   )
-  (zone (net 3) (net_name /GND) (layer B.Cu) (hatch edge 0.508)
+  (zone (net 0) (net_name "") (layer B.SilkS) (hatch full 0.508)
     (connect_pads (clearance 0.508))
     (min_thickness 0.254)
@@
     (polygon
       (pts
-        (xy 148.59 71.12) (xy 161.29 71.12) (xy 162.56 72.39) (xy 162.56 124.46) (xy 147.32 124.46)
-        (xy 142.24 119.38) (xy 142.24 109.22) (xy 147.32 104.14) (xy 147.32 72.39)
+        (xy 165.1 81.788) (xy 149.86 81.788) (xy 149.86 76.2) (xy 165.1 76.2)
       )
     )
+  )
+  (zone (net 1) (net_name /VCC) (layer F.Cu) (hatch none 0.508)
+    (connect_pads (clearance 0.508))
+    (min_thickness 0.254)
+    (fill yes (arc_segments 16) (thermal_gap 0.508) (thermal_bridge_width 0.508))
+    (polygon
+      (pts
+        (xy 165.1 72.39) (xy 165.1 137.16) (xy 147.32 137.16) (xy 147.32 124.46) (xy 144.78 121.92)
+        (xy 144.78 106.68) (xy 147.32 104.14) (xy 147.32 81.788) (xy 149.86 81.788) (xy 149.86 72.39)
+        (xy 151.13 71.12) (xy 163.83 71.12)
+      )
+    )
+  )
+  (zone (net 3) (net_name /GND) (layer B.Cu) (hatch none 0.508)
+    (connect_pads (clearance 0.508))
+    (min_thickness 0.254)
+    (fill yes (arc_segments 16) (thermal_gap 0.508) (thermal_bridge_width 0.508))
+    (polygon
+      (pts
+        (xy 165.1 72.39) (xy 165.1 137.16) (xy 147.32 137.16) (xy 147.32 124.46) (xy 144.78 121.92)
+        (xy 144.78 106.68) (xy 147.32 104.14) (xy 147.32 81.788) (xy 149.86 81.788) (xy 149.86 72.39)
+        (xy 151.13 71.12) (xy 163.83 71.12)
+      )
+    )
